File: generator.kicad_sch (KiCad schematic)
At the start: 0 parts

Commit message: Routed analog input and generator, added ethernet
Parts:
- added C3: 22p, symbol Device:C
- added C4, C7: 0.1, symbol Device:C
- added C5, C6: 220n, symbol Device:C
- added R15: 36K, symbol Device:R
- added R16, R18, R19: 10K, symbol Device:R
- added R17, R20: 470, symbol Device:R
- added U3: TSB582, Package_SO:SOIC-8-1EP_3.9x4.9mm_P1.27mm_EP2.29x3mm, symbol Amplifier_Operational:TSV912IST
Connections:
- new net: C6.2, R20.1
- new net: C3.1, R15.1, R16.2, U3.3 (+)
- new net: R18.1, R19.2, U3.5 (+)
- new net: C5.2, R17.1
- new net: C4.2, R16.1
- new net +24V: C7.2, U3.8 (V+)
- new net GIN: C4.1
- new net GND: C5.1, C6.1, C7.1, U3.4 (V-)
- new net GOUT+: C3.2, R15.2, R17.2, R19.1, U3.1
- new net GOUT-: R18.2, R20.2, U3.7
- new net VREFG: U3.2 (-), U3.6 (-)
