File: cad-enc-dec.kicad_sch (KiCad schematic)
At the start: 0 parts

Commit message: Routed analog input and generator, added ethernet
Other:
- added sheet Ethernet (ethernet.kicad_sch)
- sheet Analog Generator 1 ports: added +24V, GIN, GND, GOUT+, GOUT-, VREFG; removed none
- sheet Analog Input 1 ports: added +5V, AIN+, AIN-, AOUT, GND, VREFA; removed none
Changed lines of the file:
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@@
 (kicad_sch (version 20230121) (generator eeschema)
   (paper "A3")
-  (sheet (at 46.99 222.25) (size 25.4 25.4) (fields_autoplaced)
+  (sheet (at 90.17 121.92) (size 25.4 25.4) (fields_autoplaced)
     (stroke (width 0.1524) (type solid))
     (fill (color 0 0 0 0.0000))
-    (property "Sheetname" " Power Supply" (at 46.99 221.5384 0)
+    (property "Sheetname" " Power Supply" (at 90.17 121.2084 0)
       (effects (font (size 1.27 1.27)) (justify left bottom))
     )
-    (property "Sheetfile" "power.kicad_sch" (at 46.99 248.2346 0)
+    (property "Sheetfile" "power.kicad_sch" (at 90.17 147.9046 0)
       (effects (font (size 1.27 1.27)) (justify left top))
     )
@@
     )
   )
-  (sheet (at 127 38.1) (size 25.4 25.4) (fields_autoplaced)
+  (sheet (at 127 38.1) (size 38.1 22.86) (fields_autoplaced)
     (stroke (width 0.1524) (type solid))
     (fill (color 0 0 0 0.0000))
@@
       (effects (font (size 1.27 1.27)) (justify left bottom))
     )
-    (property "Sheetfile" "analog_in.kicad_sch" (at 127 64.0846 0)
+    (property "Sheetfile" "analog_in.kicad_sch" (at 127 61.5446 0)
       (effects (font (size 1.27 1.27)) (justify left top))
+    )
+    (pin "AIN-" input (at 127 46.99 180)
+      (effects (font (size 2.54 2.54)) (justify left))
+    )
+    (pin "AIN+" input (at 127 41.91 180)
+      (effects (font (size 2.54 2.54)) (justify left))
+    )
+    (pin "GND" input (at 165.1 46.99 0)
+      (effects (font (size 2.54 2.54)) (justify right))
+    )
+    (pin "+5V" input (at 165.1 41.91 0)
+      (effects (font (size 2.54 2.54)) (justify right))
+    )
+    (pin "AOUT" input (at 165.1 57.15 0)
+      (effects (font (size 2.54 2.54)) (justify right))
+    )
+    (pin "VREFA" input (at 127 57.15 180)
+      (effects (font (size 2.54 2.54)) (justify left))
     )
     (instances
@@
     )
   )
-  (sheet (at 203.2 38.1) (size 25.4 25.4) (fields_autoplaced)
+  (sheet (at 203.2 38.1) (size 38.1 22.86) (fields_autoplaced)
     (stroke (width 0.1524) (type solid))
     (fill (color 0 0 0 0.0000))
@@
       (effects (font (size 1.27 1.27)) (justify left bottom))
     )
-    (property "Sheetfile" "generator.kicad_sch" (at 203.2 64.0846 0)
+    (property "Sheetfile" "generator.kicad_sch" (at 203.2 61.5446 0)
       (effects (font (size 1.27 1.27)) (justify left top))
+    )
+    (pin "VREFG" input (at 203.2 57.15 180)
+      (effects (font (size 2.54 2.54)) (justify left))
+    )
+    (pin "GIN" input (at 203.2 41.91 180)
+      (effects (font (size 2.54 2.54)) (justify left))
+    )
+    (pin "+24V" input (at 241.3 41.91 0)
+      (effects (font (size 2.54 2.54)) (justify right))
+    )
+    (pin "GND" input (at 241.3 46.99 0)
+      (effects (font (size 2.54 2.54)) (justify right))
+    )
+    (pin "GOUT+" input (at 241.3 52.07 0)
+      (effects (font (size 2.54 2.54)) (justify right))
+    )
+    (pin "GOUT-" input (at 241.3 57.15 0)
+      (effects (font (size 2.54 2.54)) (justify right))
     )
     (instances
@@
     )
   )
-  (sheet (at 50.8 36.83) (size 38.1 43.18) (fields_autoplaced)
+  (sheet (at 50.8 38.1) (size 38.1 43.18) (fields_autoplaced)
     (stroke (width 0.1524) (type solid))
     (fill (color 0 0 0 0.0000))
-    (property "Sheetname" "Digital Input 1" (at 50.8 36.1184 0)
+    (property "Sheetname" "Digital Input 1" (at 50.8 37.3884 0)
       (effects (font (size 1.27 1.27)) (justify left bottom))
     )
-    (property "Sheetfile" "digital_in.kicad_sch" (at 50.8 80.5946 0)
+    (property "Sheetfile" "digital_in.kicad_sch" (at 50.8 81.8646 0)
       (effects (font (size 1.27 1.27)) (justify left top))
     )
-    (pin "DIN2-" input (at 50.8 55.88 180)
+    (pin "DIN2-" input (at 50.8 57.15 180)
       (effects (font (size 2.54 2.54)) (justify left))
     )
-    (pin "DIN2+" input (at 50.8 50.8 180)
+    (pin "DIN2+" input (at 50.8 52.07 180)
       (effects (font (size 2.54 2.54)) (justify left))
     )
-    (pin "DIN1-" input (at 50.8 45.72 180)
+    (pin "DIN1-" input (at 50.8 46.99 180)
       (effects (font (size 2.54 2.54)) (justify left))
     )
-    (pin "DIN1+" input (at 50.8 40.64 180)
+    (pin "DIN1+" input (at 50.8 41.91 180)
       (effects (font (size 2.54 2.54)) (justify left))
     )
-    (pin "DIN4-" input (at 50.8 76.2 180)
+    (pin "DIN4-" input (at 50.8 77.47 180)
       (effects (font (size 2.54 2.54)) (justify left))
     )
-    (pin "DIN3+" input (at 50.8 60.96 180)
+    (pin "DIN3+" input (at 50.8 62.23 180)
       (effects (font (size 2.54 2.54)) (justify left))
     )
-    (pin "DIN4+" input (at 50.8 71.12 180)
+    (pin "DIN4+" input (at 50.8 72.39 180)
       (effects (font (size 2.54 2.54)) (justify left))
     )
-    (pin "DIN3-" input (at 50.8 66.04 180)
+    (pin "DIN3-" input (at 50.8 67.31 180)
       (effects (font (size 2.54 2.54)) (justify left))
     )
-    (pin "DOUT4" input (at 88.9 76.2 0)
+    (pin "DOUT4" input (at 88.9 77.47 0)
       (effects (font (size 2.54 2.54)) (justify right))
     )
-    (pin "DOUT3" input (at 88.9 71.12 0)
+    (pin "DOUT3" input (at 88.9 72.39 0)
       (effects (font (size 2.54 2.54)) (justify right))
     )
-    (pin "DOUT1" input (at 88.9 60.96 0)
+    (pin "DOUT1" input (at 88.9 62.23 0)
       (effects (font (size 2.54 2.54)) (justify right))
     )
-    (pin "DOUT2" input (at 88.9 66.04 0)
+    (pin "DOUT2" input (at 88.9 67.31 0)
       (effects (font (size 2.54 2.54)) (justify right))
     )
-    (pin "GND" input (at 88.9 45.72 0)
+    (pin "GND" input (at 88.9 46.99 0)
       (effects (font (size 2.54 2.54)) (justify right))
     )
-    (pin "+5V" input (at 88.9 40.64 0)
+    (pin "+5V" input (at 88.9 41.91 0)
       (effects (font (size 2.54 2.54)) (justify right))
     )
@@
       )
     )
+  )
+  (sheet (at 152.4 114.3) (size 25.4 53.34) (fields_autoplaced)
+    (stroke (width 0.1524) (type solid))
+    (fill (color 0 0 0 0.0000))
+    (property "Sheetname" "Ethernet" (at 152.4 113.5884 0)
+      (effects (font (size 1.27 1.27)) (justify left bottom))
+    )
+    (property "Sheetfile" "ethernet.kicad_sch" (at 152.4 168.2246 0)
+      (effects (font (size 1.27 1.27)) (justify left top))
+    )
+    (pin "CRS" input (at 152.4 118.11 180)
+      (effects (font (size 2.54 2.54)) (justify left))
+    )
+    (pin "MDC" input (at 152.4 123.19 180)
+      (effects (font (size 2.54 2.54)) (justify left))
+    )
+    (pin "nINT" input (at 152.4 128.27 180)
+      (effects (font (size 2.54 2.54)) (justify left))
+    )
+    (pin "MDIO" input (at 152.4 133.35 180)
+      (effects (font (size 2.54 2.54)) (justify left))
+    )
+    (pin "nRST" input (at 152.4 138.43 180)
+      (effects (font (size 2.54 2.54)) (justify left))
+    )
+    (pin "RXD1" input (at 152.4 148.59 180)
+      (effects (font (size 2.54 2.54)) (justify left))
+    )
+    (pin "RXD0" input (at 152.4 143.51 180)
+      (effects (font (size 2.54 2.54)) (justify left))
+    )
+    (pin "TXD1" input (at 152.4 158.75 180)
+      (effects (font (size 2.54 2.54)) (justify left))
+    )
+    (pin "TXD0" input (at 152.4 153.67 180)
+      (effects (font (size 2.54 2.54)) (justify left))
+    )
+    (pin "TXEN" input (at 152.4 163.83 180)
+      (effects (font (size 2.54 2.54)) (justify left))
+    )
+    (instances
+      (project "cad-enc-dec"
+        (path "/894df1c3-1a5d-48b0-9966-84d5c2c2c705" (page "7"))
+      )
+    )

Commit message: Rearranged sheets and corrected some namings
Other:
- sheet  Power Supply renamed Power Supply 1
- sheet Analog Generator 1 renamed Analog Output 1
- removed sheet Ethernet
- added sheet Analog Input 2 (analog_in.kicad_sch)
- added sheet Analog Input 3 (analog_in.kicad_sch)
- added sheet Analog Input 4 (analog_in.kicad_sch)
- added sheet Analog Input 5 (analog_in.kicad_sch)
- added sheet Analog Input 6 (analog_in.kicad_sch)
- added sheet Analog Output 2 (analog_out.kicad_sch)
- added sheet Analog Output 3 (analog_out.kicad_sch)
- added sheet Analog Output 4 (analog_out.kicad_sch)
- added sheet Analog Output 5 (analog_out.kicad_sch)
- added sheet Analog Output 6 (analog_out.kicad_sch)
- added sheet Digital Input 2 (digital_in.kicad_sch)
- added sheet Digital Input 3 (digital_in.kicad_sch)
- added sheet Digital Input 4 (digital_in.kicad_sch)
- added sheet Digital Input 5 (digital_in.kicad_sch)
- added sheet Digital Input 6 (digital_in.kicad_sch)
- added sheet Digital Input 7 (digital_in.kicad_sch)
- added sheet Digital Input 8 (digital_in.kicad_sch)
- added sheet Digital Input 9 (digital_in.kicad_sch)
- added sheet Digital Output 1 (digital_out.kicad_sch)
- added sheet Digital Output 2 (digital_out.kicad_sch)
- added sheet Digital Output 3 (digital_out.kicad_sch)
- added sheet Digital Output 4 (digital_out.kicad_sch)
- added sheet Digital Output 5 (digital_out.kicad_sch)
- added sheet Digital Output 6 (digital_out.kicad_sch)
- added sheet Digital Output 7 (digital_out.kicad_sch)
- added sheet Digital Output 8 (digital_out.kicad_sch)
- added sheet Digital Output 9 (digital_out.kicad_sch)
- added sheet Ethernet 1 (ethernet.kicad_sch)
- added sheet Ethernet 2 (ethernet.kicad_sch)
- added sheet Power Supply 2 (power.kicad_sch)
- added sheet Receiver (receiver.kicad_sch)
- sheet Analog Input 1 ports: added VREF; removed VREFA
- sheet Analog Output 1: file generator.kicad_sch -> analog_out.kicad_sch
- sheet Analog Output 1 ports: added AIN, AOUT+, AOUT-, VREF; removed GIN, GOUT+, GOUT-, VREFG
- sheet Digital Input 1 ports: added +3V3; removed +5V

Commit message: Updated boards hierarchy
Other:
- removed sheet Analog Input 1
- removed sheet Analog Input 2
- removed sheet Analog Input 3
- removed sheet Analog Input 4
- removed sheet Analog Input 5
- removed sheet Analog Input 6
- removed sheet Analog Output 1
- removed sheet Analog Output 2
- removed sheet Analog Output 3
- removed sheet Analog Output 4
- removed sheet Analog Output 5
- removed sheet Analog Output 6
- removed sheet Digital Input 1
- removed sheet Digital Input 2
- removed sheet Digital Input 3
- removed sheet Digital Input 4
- removed sheet Digital Input 5
- removed sheet Digital Input 6
- removed sheet Digital Input 7
- removed sheet Digital Input 8
- removed sheet Digital Input 9
- removed sheet Digital Output 1
- removed sheet Digital Output 2
- removed sheet Digital Output 3
- removed sheet Digital Output 4
- removed sheet Digital Output 5
- removed sheet Digital Output 6
- removed sheet Digital Output 7
- removed sheet Digital Output 8
- removed sheet Digital Output 9
- removed sheet Ethernet 1
- removed sheet Ethernet 2
- removed sheet Power Supply 1
- removed sheet Power Supply 2
- removed sheet Receiver
- removed sheet Transmitter
- added sheet Analog Board (analog.kicad_sch)
- added sheet Input Board (input.kicad_sch)
- added sheet Output Board (output.kicad_sch)
