File: input.kicad_sch (KiCad schematic)
At the start: 6 parts, among them J3 Conn_02x06_Odd_Even, J4 Conn_02x06_Odd_Even, J5 Conn_02x06_Odd_Even, J6 Conn_02x06_Odd_Even, J7 Conn_02x06_Odd_Even, J8 Conn_02x06_Odd_Even

Commit message: Finished annotation
Parts:
- added J205: Conn_01x04, symbol Connector_Generic:Conn_01x04
- added J206: Conn_02x12_Odd_Even, symbol Connector_Generic:Conn_02x12_Odd_Even
- renumbered J3 to J201, J4 to J202, J5 to J203, J6 to J204, J7 to J207, J8 to J208
Connections:
- new net +24V: J206.2 (Pin_2)
- new net +5V: J205.1 (Pin_1), J206.1 (Pin_1)
- new net GIN: J206.3 (Pin_3), J206.4 (Pin_4), J206.5 (Pin_5), J206.6 (Pin_6), J206.7 (Pin_7), J206.8 (Pin_8)
- new net GND: J205.4 (Pin_4), J206.23 (Pin_23), J206.24 (Pin_24)
- new net RE1_COS: J206.10 (Pin_10)
- new net RE1_SIN: J206.9 (Pin_9)
- new net RE2_COS: J206.12 (Pin_12)
- new net RE2_SIN: J206.11 (Pin_11)
- new net RE3_COS: J206.14 (Pin_14)
- new net RE3_SIN: J206.13 (Pin_13)
- new net RE4_COS: J206.16 (Pin_16)
- new net RE4_SIN: J206.15 (Pin_15)
- new net RE5_COS: J206.18 (Pin_18)
- new net RE5_SIN: J206.17 (Pin_17)
- new net RE6_COS: J206.20 (Pin_20)
- new net RE6_SIN: J206.19 (Pin_19)
- new net SWDCLK: J205.3 (Pin_3)
- new net SWDIO: J205.2 (Pin_2)
- new net VREF: J206.21 (Pin_21), J206.22 (Pin_22)
Other:
- sheet Digital Input 1 ports: added DIN1, DIN2, DIN3, DIN4; removed DOUT1, DOUT2, DOUT3, DOUT4
- sheet Digital Input 2 ports: added DIN1, DIN2, DIN3, DIN4; removed DOUT1, DOUT2, DOUT3, DOUT4
- sheet Digital Input 3 ports: added DIN1, DIN2, DIN3, DIN4; removed DOUT1, DOUT2, DOUT3, DOUT4
- sheet Digital Input 4 ports: added DIN1, DIN2, DIN3, DIN4; removed DOUT1, DOUT2, DOUT3, DOUT4
- sheet Digital Input 5 ports: added DIN1, DIN2, DIN3, DIN4; removed DOUT1, DOUT2, DOUT3, DOUT4
- sheet Digital Input 6 ports: added DIN1, DIN2, DIN3, DIN4; removed DOUT1, DOUT2, DOUT3, DOUT4
- sheet Digital Input 7 ports: added DIN1, DIN2, DIN3, DIN4; removed DOUT1, DOUT2, DOUT3, DOUT4
- sheet Digital Input 8 ports: added DIN1, DIN2, DIN3, DIN4; removed DOUT1, DOUT2, DOUT3, DOUT4
- sheet Digital Input 9 ports: added DIN1, DIN2, DIN3, DIN4; removed DOUT1, DOUT2, DOUT3, DOUT4
- sheet Ethernet 1 ports: added REFCLK; removed +3V3, GND, nINT
- sheet Transmitter ports: added AIN1_1, AIN1_2, AIN2_1, AIN2_2, AIN3_1, AIN3_2, AIN4_1, AIN4_2, AIN5_1, AIN5_2, AIN6_1, AIN6_2, DIN1_1, DIN1_2, DIN1_3, DIN1_4, DIN1_5, DIN1_6, DIN2_1, DIN2_2, DIN2_3, DIN2_4, DIN2_5, DIN2_6, DIN3_1, DIN3_2, DIN3_3, DIN3_4, DIN3_5, DIN3_6, DIN4_1, DIN4_2, DIN4_3, DIN4_4, DIN4_5, DIN4_6, DIN5_1, DIN5_2, DIN5_3, DIN5_4, DIN5_5, DIN5_6, DIN6_1, DIN6_2, DIN6_3, DIN6_4, DIN6_5, DIN6_6, ETH_CRS, ETH_MDC, ETH_MDIO, ETH_NRST, ETH_REFCLK, ETH_RXD0, ETH_RXD1, ETH_TXD0, ETH_TXD1, ETH_TXEN, GENOUT, SWD_CLK, SWD_IO, VREF; removed none

Commit message: Merged receiver and transmitter
Parts:
- added J206: Conn_02x06_Odd_Even, symbol Connector_Generic:Conn_02x06_Odd_Even
- renumbered J206 to J207, J207 to J208, J208 to J209
Connections:
- net +5V: now also J206.1 (Pin_1), J206.11 (Pin_11), J206.3 (Pin_3), J206.5 (Pin_5), J206.7 (Pin_7), J206.9 (Pin_9); no longer J205.1 (Pin_1)
- net GND: now also J206.10 (Pin_10), J206.12 (Pin_12), J206.2 (Pin_2), J206.4 (Pin_4), J206.6 (Pin_6), J206.8 (Pin_8)
- net SWDCLK: now also J205.2 (Pin_2); no longer J205.3 (Pin_3)
- net SWDIO: now also J205.3 (Pin_3); no longer J205.2 (Pin_2)
- net GIN renamed GENOUT
- net VREF renamed VREFOUT
- new net +3V3: J205.1 (Pin_1)
Other:
- sheet Digital Input 1 ports: added none; removed +3V3, GND
- sheet Digital Input 2 ports: added none; removed +3V3, GND
- sheet Digital Input 3 ports: added none; removed +3V3, GND
- sheet Digital Input 4 ports: added none; removed +3V3, GND
- sheet Digital Input 5 ports: added none; removed +3V3, GND
- sheet Digital Input 6 ports: added none; removed +3V3, GND
- sheet Digital Input 7 ports: added none; removed +3V3, GND
- sheet Digital Input 8 ports: added none; removed +3V3, GND
- sheet Digital Input 9 ports: added none; removed +3V3, GND
- sheet Transmitter: file transmitter.kicad_sch -> serializer.kicad_sch
- sheet Transmitter ports: added GEN, GPIO1_1, GPIO1_2, GPIO1_3, GPIO1_4, GPIO1_5, GPIO1_6, GPIO2_1, GPIO2_2, GPIO2_3, GPIO2_4, GPIO2_5, GPIO2_6, GPIO3_1, GPIO3_2, GPIO3_3, GPIO3_4, GPIO3_5, GPIO3_6, GPIO4_1, GPIO4_2, GPIO4_3, GPIO4_4, GPIO4_5, GPIO4_6, GPIO5_1, GPIO5_2, GPIO5_3, GPIO5_4, GPIO5_5, GPIO5_6, GPIO6_1, GPIO6_2, GPIO6_3, GPIO6_4, GPIO6_5, GPIO6_6; removed DIN1_1, DIN1_2, DIN1_3, DIN1_4, DIN1_5, DIN1_6, DIN2_1, DIN2_2, DIN2_3, DIN2_4, DIN2_5, DIN2_6, DIN3_1, DIN3_2, DIN3_3, DIN3_4, DIN3_5, DIN3_6, DIN4_1, DIN4_2, DIN4_3, DIN4_4, DIN4_5, DIN4_6, DIN5_1, DIN5_2, DIN5_3, DIN5_4, DIN5_5, DIN5_6, DIN6_1, DIN6_2, DIN6_3, DIN6_4, DIN6_5, DIN6_6, GENOUT
- moved on the sheet: J205, J207
