File: output.kicad_sch (KiCad schematic)
At the start: 6 parts, among them J10 Conn_02x06_Odd_Even, J11 Conn_02x06_Odd_Even, J12 Conn_02x06_Odd_Even, J13 Conn_02x06_Odd_Even, J14 Conn_02x06_Odd_Even, J9 Conn_02x06_Odd_Even

Commit message: Finished annotation
Parts:
- added J605: Conn_01x04, symbol Connector_Generic:Conn_01x04
- renumbered J9 to J601, J10 to J602, J11 to J603, J12 to J604, J13 to J606, J14 to J607
Connections:
- new net +5V: J605.1 (Pin_1)
- new net GND: J605.4 (Pin_4)
- new net SWDCLK: J605.3 (Pin_3)
- new net SWDIO: J605.2 (Pin_2)
Other:
- sheet Digital Output 1 ports: added DIN1+, DIN1-, DIN2+, DIN2-, DIN3+, DIN3-, DIN4+, DIN4-; removed DOUT1+, DOUT1-, DOUT2+, DOUT2-, DOUT3+, DOUT3-, DOUT4+, DOUT4-
- sheet Digital Output 2 ports: added DIN1+, DIN1-, DIN2+, DIN2-, DIN3+, DIN3-, DIN4+, DIN4-; removed DOUT1+, DOUT1-, DOUT2+, DOUT2-, DOUT3+, DOUT3-, DOUT4+, DOUT4-
- sheet Digital Output 3 ports: added DIN1+, DIN1-, DIN2+, DIN2-, DIN3+, DIN3-, DIN4+, DIN4-; removed DOUT1+, DOUT1-, DOUT2+, DOUT2-, DOUT3+, DOUT3-, DOUT4+, DOUT4-
- sheet Digital Output 4 ports: added DIN1+, DIN1-, DIN2+, DIN2-, DIN3+, DIN3-, DIN4+, DIN4-; removed DOUT1+, DOUT1-, DOUT2+, DOUT2-, DOUT3+, DOUT3-, DOUT4+, DOUT4-
- sheet Digital Output 5 ports: added DIN1+, DIN1-, DIN2+, DIN2-, DIN3+, DIN3-, DIN4+, DIN4-; removed DOUT1+, DOUT1-, DOUT2+, DOUT2-, DOUT3+, DOUT3-, DOUT4+, DOUT4-
- sheet Digital Output 6 ports: added DIN1+, DIN1-, DIN2+, DIN2-, DIN3+, DIN3-, DIN4+, DIN4-; removed DOUT1+, DOUT1-, DOUT2+, DOUT2-, DOUT3+, DOUT3-, DOUT4+, DOUT4-
- sheet Digital Output 7 ports: added DIN1+, DIN1-, DIN2+, DIN2-, DIN3+, DIN3-, DIN4+, DIN4-; removed DOUT1+, DOUT1-, DOUT2+, DOUT2-, DOUT3+, DOUT3-, DOUT4+, DOUT4-
- sheet Digital Output 8 ports: added DIN1+, DIN1-, DIN2+, DIN2-, DIN3+, DIN3-, DIN4+, DIN4-; removed DOUT1+, DOUT1-, DOUT2+, DOUT2-, DOUT3+, DOUT3-, DOUT4+, DOUT4-
- sheet Digital Output 9 ports: added DIN1+, DIN1-, DIN2+, DIN2-, DIN3+, DIN3-, DIN4+, DIN4-; removed DOUT1+, DOUT1-, DOUT2+, DOUT2-, DOUT3+, DOUT3-, DOUT4+, DOUT4-
- sheet Ethernet 2 ports: added REFCLK; removed +3V3, GND, nINT
- sheet Receiver ports: added DOUT1_1, DOUT1_2, DOUT1_3, DOUT1_4, DOUT1_5, DOUT1_6, DOUT2_1, DOUT2_2, DOUT2_3, DOUT2_4, DOUT2_5, DOUT2_6, DOUT3_1, DOUT3_2, DOUT3_3, DOUT3_4, DOUT3_5, DOUT3_6, DOUT4_1, DOUT4_2, DOUT4_3, DOUT4_4, DOUT4_5, DOUT4_6, DOUT5_1, DOUT5_2, DOUT5_3, DOUT5_4, DOUT5_5, DOUT5_6, DOUT6_1, DOUT6_2, DOUT6_3, DOUT6_4, DOUT6_5, DOUT6_6, ETH_CRS, ETH_MDC, ETH_MDIO, ETH_NRST, ETH_REFCLK, ETH_RXD0, ETH_RXD1, ETH_TXD0, ETH_TXD1, ETH_TXEN, SWD_CLK, SWD_IO; removed none

Commit message: Merged receiver and transmitter
Parts:
- added J606: Conn_02x06_Odd_Even, symbol Connector_Generic:Conn_02x06_Odd_Even
- added J607: Conn_02x12_Odd_Even, symbol Connector_Generic:Conn_02x12_Odd_Even
- renumbered J606 to J608, J607 to J609
Connections:
- net +5V: now also J606.1 (Pin_1), J606.11 (Pin_11), J606.3 (Pin_3), J606.5 (Pin_5), J606.7 (Pin_7), J606.9 (Pin_9), J607.1 (Pin_1); no longer J605.1 (Pin_1)
- net GND: now also J606.10 (Pin_10), J606.12 (Pin_12), J606.2 (Pin_2), J606.4 (Pin_4), J606.6 (Pin_6), J606.8 (Pin_8), J607.23 (Pin_23), J607.24 (Pin_24)
- new net +24V: J607.2 (Pin_2)
- new net +3.3V: J605.1 (Pin_1)
- new net GENOUT: J607.3 (Pin_3), J607.4 (Pin_4), J607.5 (Pin_5), J607.6 (Pin_6), J607.7 (Pin_7), J607.8 (Pin_8)
- new net RE1_COS: J607.10 (Pin_10)
- new net RE1_SIN: J607.9 (Pin_9)
- new net RE2_COS: J607.12 (Pin_12)
- new net RE2_SIN: J607.11 (Pin_11)
- new net RE3_COS: J607.14 (Pin_14)
- new net RE3_SIN: J607.13 (Pin_13)
- new net RE4_COS: J607.16 (Pin_16)
- new net RE4_SIN: J607.15 (Pin_15)
- new net RE5_COS: J607.18 (Pin_18)
- new net RE5_SIN: J607.17 (Pin_17)
- new net RE6_COS: J607.20 (Pin_20)
- new net RE6_SIN: J607.19 (Pin_19)
- new net VREFOUT: J607.21 (Pin_21), J607.22 (Pin_22)
Other:
- sheet Digital Output 1 ports: added DOUT1, DOUT1+, DOUT1-, DOUT2, DOUT2+, DOUT2-, DOUT3, DOUT3+, DOUT3-, DOUT4, DOUT4+, DOUT4-; removed +5V, DIN1, DIN1+, DIN1-, DIN2, DIN2+, DIN2-, DIN3, DIN3+, DIN3-, DIN4, DIN4+, DIN4-, GND
- sheet Digital Output 2 ports: added DOUT1, DOUT1+, DOUT1-, DOUT2, DOUT2+, DOUT2-, DOUT3, DOUT3+, DOUT3-, DOUT4, DOUT4+, DOUT4-; removed +5V, DIN1, DIN1+, DIN1-, DIN2, DIN2+, DIN2-, DIN3, DIN3+, DIN3-, DIN4, DIN4+, DIN4-, GND
- sheet Digital Output 3 ports: added DOUT1, DOUT1+, DOUT1-, DOUT2, DOUT2+, DOUT2-, DOUT3, DOUT3+, DOUT3-, DOUT4, DOUT4+, DOUT4-; removed +5V, DIN1, DIN1+, DIN1-, DIN2, DIN2+, DIN2-, DIN3, DIN3+, DIN3-, DIN4, DIN4+, DIN4-, GND
- sheet Digital Output 4 ports: added DOUT1, DOUT1+, DOUT1-, DOUT2, DOUT2+, DOUT2-, DOUT3, DOUT3+, DOUT3-, DOUT4, DOUT4+, DOUT4-; removed +5V, DIN1, DIN1+, DIN1-, DIN2, DIN2+, DIN2-, DIN3, DIN3+, DIN3-, DIN4, DIN4+, DIN4-, GND
- sheet Digital Output 5 ports: added DOUT1, DOUT1+, DOUT1-, DOUT2, DOUT2+, DOUT2-, DOUT3, DOUT3+, DOUT3-, DOUT4, DOUT4+, DOUT4-; removed +5V, DIN1, DIN1+, DIN1-, DIN2, DIN2+, DIN2-, DIN3, DIN3+, DIN3-, DIN4, DIN4+, DIN4-, GND
- sheet Digital Output 6 ports: added DOUT1, DOUT1+, DOUT1-, DOUT2, DOUT2+, DOUT2-, DOUT3, DOUT3+, DOUT3-, DOUT4, DOUT4+, DOUT4-; removed +5V, DIN1, DIN1+, DIN1-, DIN2, DIN2+, DIN2-, DIN3, DIN3+, DIN3-, DIN4, DIN4+, DIN4-, GND
- sheet Digital Output 7 ports: added DOUT1, DOUT1+, DOUT1-, DOUT2, DOUT2+, DOUT2-, DOUT3, DOUT3+, DOUT3-, DOUT4, DOUT4+, DOUT4-; removed +5V, DIN1, DIN1+, DIN1-, DIN2, DIN2+, DIN2-, DIN3, DIN3+, DIN3-, DIN4, DIN4+, DIN4-, GND
- sheet Digital Output 8 ports: added DOUT1, DOUT1+, DOUT1-, DOUT2, DOUT2+, DOUT2-, DOUT3, DOUT3+, DOUT3-, DOUT4, DOUT4+, DOUT4-; removed +5V, DIN1, DIN1+, DIN1-, DIN2, DIN2+, DIN2-, DIN3, DIN3+, DIN3-, DIN4, DIN4+, DIN4-, GND
- sheet Digital Output 9 ports: added DOUT1, DOUT1+, DOUT1-, DOUT2, DOUT2+, DOUT2-, DOUT3, DOUT3+, DOUT3-, DOUT4, DOUT4+, DOUT4-; removed +5V, DIN1, DIN1+, DIN1-, DIN2, DIN2+, DIN2-, DIN3, DIN3+, DIN3-, DIN4, DIN4+, DIN4-, GND
- sheet Receiver: file receiver.kicad_sch -> serializer.kicad_sch
- sheet Receiver ports: added AIN1_1, AIN1_2, AIN2_1, AIN2_2, AIN3_1, AIN3_2, AIN4_1, AIN4_2, AIN5_1, AIN5_2, AIN6_1, AIN6_2, GEN, GPIO1_1, GPIO1_2, GPIO1_3, GPIO1_4, GPIO1_5, GPIO1_6, GPIO2_1, GPIO2_2, GPIO2_3, GPIO2_4, GPIO2_5, GPIO2_6, GPIO3_1, GPIO3_2, GPIO3_3, GPIO3_4, GPIO3_5, GPIO3_6, GPIO4_1, GPIO4_2, GPIO4_3, GPIO4_4, GPIO4_5, GPIO4_6, GPIO5_1, GPIO5_2, GPIO5_3, GPIO5_4, GPIO5_5, GPIO5_6, GPIO6_1, GPIO6_2, GPIO6_3, GPIO6_4, GPIO6_5, GPIO6_6, VREF; removed DOUT1_1, DOUT1_2, DOUT1_3, DOUT1_4, DOUT1_5, DOUT1_6, DOUT2_1, DOUT2_2, DOUT2_3, DOUT2_4, DOUT2_5, DOUT2_6, DOUT3_1, DOUT3_2, DOUT3_3, DOUT3_4, DOUT3_5, DOUT3_6, DOUT4_1, DOUT4_2, DOUT4_3, DOUT4_4, DOUT4_5, DOUT4_6, DOUT5_1, DOUT5_2, DOUT5_3, DOUT5_4, DOUT5_5, DOUT5_6, DOUT6_1, DOUT6_2, DOUT6_3, DOUT6_4, DOUT6_5, DOUT6_6
- moved on the sheet: J605

Commit message: Fixed ERC errors and warnings
Connections:
- net +3.3V renamed +3V3
Changed lines of the file:
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@@
     (effects (font (size 1.27 1.27)) (justify right bottom))
+  )
+  (symbol (lib_id "power:+3V3") (at 93.98 453.39 0) (unit 1)
+    (in_bom yes) (on_board yes) (dnp no) (fields_autoplaced)
+    (property "Reference" "#PWR0601" (at 93.98 457.2 0)
+      (effects (font (size 1.27 1.27)) hide)
+    )
+    (property "Value" "+3V3" (at 93.98 448.31 0)
+      (effects (font (size 1.27 1.27)))
+    )
+    (property "Footprint" "" (at 93.98 453.39 0)
+      (effects (font (size 1.27 1.27)) hide)
+    )
+    (property "Datasheet" "" (at 93.98 453.39 0)
+      (effects (font (size 1.27 1.27)) hide)
+    )
+    (pin "1")
+    (instances
+      (project "cad-enc-dec"
+        (path "/894df1c3-1a5d-48b0-9966-84d5c2c2c705/0815129a-f835-434b-a91c-b449ee32428d"
+          (reference "#PWR0601") (unit 1)
+        )
+      )
+    )
   )
   (symbol (lib_id "Connector_Generic:Conn_02x12_Odd_Even") (at 106.68 560.07 0) (unit 1)
@@
         )
       )
-    )
-  )
-  (symbol (lib_id "power:+3.3V") (at 93.98 453.39 0) (unit 1)
-    (in_bom yes) (on_board yes) (dnp no) (fields_autoplaced)
-    (property "Reference" "#PWR0601" (at 93.98 457.2 0)
-      (effects (font (size 1.27 1.27)) hide)
-    )
-    (property "Value" "+3.3V" (at 93.98 448.31 0)
-      (effects (font (size 1.27 1.27)))
-    )
-    (property "Footprint" "" (at 93.98 453.39 0)
-      (effects (font (size 1.27 1.27)) hide)
-    )
-    (property "Datasheet" "" (at 93.98 453.39 0)
-      (effects (font (size 1.27 1.27)) hide)
-    )
-    (pin "1")
-    (instances
-      (project "cad-enc-dec"
-        (path "/894df1c3-1a5d-48b0-9966-84d5c2c2c705/0815129a-f835-434b-a91c-b449ee32428d"
-          (reference "#PWR0601") (unit 1)
-        )
-      )
