File: analog_in.kicad_sch (KiCad schematic)
At the start: 9 parts, among them U3301 INA600B, U3302 CDSOT236-T12, U3303 INA600B

Commit message: Split schematic into three subprojects
Parts:
- renumbered C3301 to C11, C3302 to C12, R3301 to R21, R3302 to R22, R3303 to R23, R3304 to R24, U3301 to U16, U3302 to U17, U3303 to U18

Commit message: Assigned footprints for analog circuit
Parts:
- C11, C12: value 100n -> 100nF
- U17: value CDSOT236-T12 -> TPCDSOT236-T12
Changed lines of the file:
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@@
       (effects (font (size 1.27 1.27)) (justify left))
     )
-    (property "Value" "CDSOT236-T12" (at 147.32 81.28 0)
+    (property "Value" "TPCDSOT236-T12" (at 147.32 81.28 0)
       (effects (font (size 1.27 1.27)) (justify left))
     )
@@
       (effects (font (size 1.27 1.27)) hide)
     )
-    (property "Datasheet" "https://www.bourns.com/docs/product-datasheets/cdsot236-0504c.pdf" (at 154.94 97.79 0)
+    (property "Datasheet" "https://www.lcsc.com/product-detail/C48543240.html" (at 154.94 97.79 0)
       (effects (font (size 1.27 1.27)) hide)
     )
@@
   )
   (symbol (lib_id "Amplifier_Current:INA181") (at 198.12 59.69 0) (unit 1)
-    (in_bom yes) (on_board yes) (dnp no) (fields_autoplaced)
-    (property "Reference" "U16" (at 208.28 55.4991 0)
-      (effects (font (size 1.27 1.27)))
-    )
-    (property "Value" "INA600B" (at 208.28 58.0391 0)
+    (in_bom yes) (on_board yes) (dnp no)
+    (property "Reference" "U16" (at 201.93 53.34 0)
+      (effects (font (size 1.27 1.27)))
+    )
+    (property "Value" "INA600B" (at 201.93 55.88 0)
       (effects (font (size 1.27 1.27)))
     )
@@
       (effects (font (size 1.27 1.27)) hide)
     )
-    (property "Datasheet" "" (at 201.93 55.88 0)
+    (property "Datasheet" "https://www.lcsc.com/product-detail/C51890378.html" (at 201.93 55.88 0)
       (effects (font (size 1.27 1.27)) hide)
     )
@@
   (symbol (lib_id "Device:R") (at 124.46 57.15 90) (unit 1)
     (in_bom yes) (on_board yes) (dnp no)
-    (property "Reference" "R21" (at 124.46 50.8 90)
-      (effects (font (size 1.27 1.27)) hide)
+    (property "Reference" "R21" (at 124.46 55.118 90)
+      (effects (font (size 1.27 1.27)))
     )
     (property "Value" "100" (at 124.46 57.15 90)
@@
       (effects (font (size 1.27 1.27)) hide)
     )
-    (property "Datasheet" "~" (at 124.46 57.15 0)
+    (property "Datasheet" "100Ω 75V Thick Film 1%" (at 124.46 57.15 0)
       (effects (font (size 1.27 1.27)) hide)
     )
@@
   (symbol (lib_id "Device:R") (at 124.46 130.81 90) (unit 1)
     (in_bom yes) (on_board yes) (dnp no)
-    (property "Reference" "R23" (at 124.46 124.46 90)
-      (effects (font (size 1.27 1.27)) hide)
+    (property "Reference" "R23" (at 124.46 128.778 90)
+      (effects (font (size 1.27 1.27)))
     )
     (property "Value" "100" (at 124.46 130.81 90)
@@
       (effects (font (size 1.27 1.27)) hide)
     )
-    (property "Datasheet" "~" (at 124.46 130.81 0)
+    (property "Datasheet" "100Ω 75V Thick Film 1%" (at 124.46 130.81 0)
       (effects (font (size 1.27 1.27)) hide)
     )
@@
       (effects (font (size 1.27 1.27)))
     )
-    (property "Value" "100n" (at 189.23 109.22 90)
+    (property "Value" "100nF" (at 189.23 109.22 90)
       (effects (font (size 1.27 1.27)))
     )
@@
       (effects (font (size 1.27 1.27)) hide)
     )
-    (property "Datasheet" "~" (at 189.23 114.3 0)
+    (property "Datasheet" "100nF 50V X7R 10%" (at 189.23 114.3 0)
       (effects (font (size 1.27 1.27)) hide)
     )
@@
   )
   (symbol (lib_id "Amplifier_Current:INA181") (at 198.12 133.35 0) (unit 1)
-    (in_bom yes) (on_board yes) (dnp no) (fields_autoplaced)
-    (property "Reference" "U18" (at 208.28 129.1591 0)
-      (effects (font (size 1.27 1.27)))
-    )
-    (property "Value" "INA600B" (at 208.28 131.6991 0)
+    (in_bom yes) (on_board yes) (dnp no)
+    (property "Reference" "U18" (at 201.93 127 0)
+      (effects (font (size 1.27 1.27)))
+    )
+    (property "Value" "INA600B" (at 201.93 129.54 0)
       (effects (font (size 1.27 1.27)))
     )
@@
       (effects (font (size 1.27 1.27)) hide)
     )
-    (property "Datasheet" "" (at 201.93 129.54 0)
+    (property "Datasheet" "https://www.lcsc.com/product-detail/C51890378.html" (at 201.93 129.54 0)
       (effects (font (size 1.27 1.27)) hide)
     )
@@
       (effects (font (size 1.27 1.27)))
     )
-    (property "Value" "100n" (at 189.23 35.56 90)
+    (property "Value" "100nF" (at 189.23 35.56 90)
       (effects (font (size 1.27 1.27)))
     )
@@
       (effects (font (size 1.27 1.27)) hide)
     )
-    (property "Datasheet" "~" (at 189.23 40.64 0)
+    (property "Datasheet" "100nF 50V X7R 10%" (at 189.23 40.64 0)
       (effects (font (size 1.27 1.27)) hide)
     )
@@
   (symbol (lib_id "Device:R") (at 124.46 62.23 90) (unit 1)
     (in_bom yes) (on_board yes) (dnp no)
-    (property "Reference" "R22" (at 124.46 55.88 90)
-      (effects (font (size 1.27 1.27)) hide)
+    (property "Reference" "R22" (at 124.46 60.198 90)
+      (effects (font (size 1.27 1.27)))
     )
     (property "Value" "100" (at 124.46 62.23 90)
@@
       (effects (font (size 1.27 1.27)) hide)
     )
-    (property "Datasheet" "~" (at 124.46 62.23 0)
+    (property "Datasheet" "100Ω 75V Thick Film 1%" (at 124.46 62.23 0)
       (effects (font (size 1.27 1.27)) hide)
     )
@@
   (symbol (lib_id "Device:R") (at 124.46 135.89 90) (unit 1)
     (in_bom yes) (on_board yes) (dnp no)
-    (property "Reference" "R24" (at 124.46 129.54 90)
-      (effects (font (size 1.27 1.27)) hide)
+    (property "Reference" "R24" (at 124.46 133.858 90)
+      (effects (font (size 1.27 1.27)))
     )
     (property "Value" "100" (at 124.46 135.89 90)
@@
       (effects (font (size 1.27 1.27)) hide)
     )
-    (property "Datasheet" "~" (at 124.46 135.89 0)
-      (effects (font (size 1.27 1.27)) hide)
-    )
+    (property "Datasheet" "100Ω 75V Thick Film 1%" (at 124.46 135.89 0)
+      (effects (font (size 1.27 1.27)) hide)
+    )

Commit message: Updated files to kicad 10
Parts:
- renumbered C11 to C1, C12 to C2, R21 to R1, R22 to R2, R23 to R3, R24 to R4, U16 to U1, U17 to U2, U18 to U3
Other:
- moved on the sheet: C1, C2, R1, R2, R3, R4, U1, U2, U3
