File: digital_in.kicad_sch (KiCad schematic)
At the start: 20 parts, among them U23 SRV05-4, U24 AM26LV32E, U25 SRV05-4

Commit message: Redone power input circuit
Parts:
- renumbered C43 to C45, R123 to R122, R124 to R123, R127 to R126, R128 to R127, R131 to R130, R132 to R131, R135 to R134, R136 to R135, R26 to R25, R29 to R28, R30 to R29, R33 to R32, R34 to R33, R37 to R36, R38 to R37, R41 to R40, U23 to U24, U24 to U25, U25 to U26

Commit message: Optimized components by cost and footprint size
Parts:
- renumbered C45 to C43, R122 to R121, R126 to R122, R130 to R123, R134 to R124, R123 to R133, R127 to R134, R131 to R135, R135 to R136, R25 to R29, R28 to R30, R29 to R31, R36 to R34, R37 to R35, R40 to R36, U24 to U23, U26 to U24

Commit message: Excluded rare components
Parts:
- renumbered R121 to R123, R122 to R124, R123 to R125, R124 to R126, R133 to R135, R134 to R136, R135 to R137, R136 to R138, R29 to R31, R30 to R32, R31 to R33, R32 to R34, R33 to R35, R34 to R36, R35 to R37, R36 to R38

Commit message: Updated files to kicad 10
Parts:
- renumbered C43 to C37, R123 to R27, R124 to R28, R125 to R29, R126 to R30, R135 to R39, R136 to R40, R137 to R41, R138 to R42, U23 to U5, U24 to U6, U25 to U7
