File: digital_out.kicad_sch (KiCad schematic)
At the start: 20 parts, among them U20 CDSOT236-T05, U21 AM26LV31E, U22 CDSOT236-T05

Commit message: Set capacitor and resistor values on tranciever circuits
Parts:
- C42: value 100n -> 100nF
- R106, R108, R110, R112, R115, R116, R119, R120: value 0 -> 0R
Changed lines of the file:
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@@
       (effects (font (size 1.27 1.27)))
     )
-    (property "Value" "0" (at 146.05 101.6 90)
+    (property "Value" "0R" (at 146.05 101.6 90)
       (effects (font (size 1.27 1.27)))
     )
@@
       (effects (font (size 1.27 1.27)) hide)
     )
-    (property "Datasheet" "~" (at 146.05 101.6 0)
+    (property "Datasheet" "0Ω 75V Thick Film 1%" (at 146.05 101.6 0)
       (effects (font (size 1.27 1.27)) hide)
     )
@@
       (effects (font (size 1.27 1.27)))
     )
-    (property "Value" "0" (at 92.71 109.22 90)
+    (property "Value" "0R" (at 92.71 109.22 90)
       (effects (font (size 1.27 1.27)))
     )
@@
       (effects (font (size 1.27 1.27)) hide)
     )
-    (property "Datasheet" "~" (at 92.71 109.22 0)
+    (property "Datasheet" "0Ω 75V Thick Film 1%" (at 92.71 109.22 0)
       (effects (font (size 1.27 1.27)) hide)
     )
@@
       (effects (font (size 1.27 1.27)) hide)
     )
-    (property "Datasheet" "~" (at 209.55 81.28 0)
+    (property "Datasheet" "10Ω 75V Thick Film 1%" (at 209.55 81.28 0)
       (effects (font (size 1.27 1.27)) hide)
     )
@@
       (effects (font (size 1.27 1.27)))
     )
-    (property "Value" "0" (at 92.71 81.28 90)
+    (property "Value" "0R" (at 92.71 81.28 90)
       (effects (font (size 1.27 1.27)))
     )
@@
       (effects (font (size 1.27 1.27)) hide)
     )
-    (property "Datasheet" "~" (at 92.71 81.28 0)
+    (property "Datasheet" "0Ω 75V Thick Film 1%" (at 92.71 81.28 0)
       (effects (font (size 1.27 1.27)) hide)
     )
@@
       (effects (font (size 1.27 1.27)))
     )
-    (property "Value" "0" (at 146.05 83.82 90)
+    (property "Value" "0R" (at 146.05 83.82 90)
       (effects (font (size 1.27 1.27)))
     )
@@
       (effects (font (size 1.27 1.27)) hide)
     )
-    (property "Datasheet" "~" (at 146.05 83.82 0)
+    (property "Datasheet" "0Ω 75V Thick Film 1%" (at 146.05 83.82 0)
       (effects (font (size 1.27 1.27)) hide)
     )
@@
       (effects (font (size 1.27 1.27)))
     )
-    (property "Value" "0" (at 92.71 73.66 90)
+    (property "Value" "0R" (at 92.71 73.66 90)
       (effects (font (size 1.27 1.27)))
     )
@@
       (effects (font (size 1.27 1.27)) hide)
     )
-    (property "Datasheet" "~" (at 92.71 73.66 0)
+    (property "Datasheet" "0Ω 75V Thick Film 1%" (at 92.71 73.66 0)
       (effects (font (size 1.27 1.27)) hide)
     )
@@
       (effects (font (size 1.27 1.27)))
     )
-    (property "Value" "0" (at 146.05 76.2 90)
+    (property "Value" "0R" (at 146.05 76.2 90)
       (effects (font (size 1.27 1.27)))
     )
@@
       (effects (font (size 1.27 1.27)) hide)
     )
-    (property "Datasheet" "~" (at 146.05 76.2 0)
+    (property "Datasheet" "0Ω 75V Thick Film 1%" (at 146.05 76.2 0)
       (effects (font (size 1.27 1.27)) hide)
     )
@@
       (effects (font (size 1.27 1.27)))
     )
-    (property "Value" "0" (at 146.05 109.22 90)
+    (property "Value" "0R" (at 146.05 109.22 90)
       (effects (font (size 1.27 1.27)))
     )
@@
       (effects (font (size 1.27 1.27)) hide)
     )
-    (property "Datasheet" "~" (at 146.05 109.22 0)
+    (property "Datasheet" "0Ω 75V Thick Film 1%" (at 146.05 109.22 0)
       (effects (font (size 1.27 1.27)) hide)
     )
@@
       (effects (font (size 1.27 1.27)) hide)
     )
-    (property "Datasheet" "~" (at 209.55 101.6 0)
+    (property "Datasheet" "10Ω 75V Thick Film 1%" (at 209.55 101.6 0)
       (effects (font (size 1.27 1.27)) hide)
     )
@@
       (effects (font (size 1.27 1.27)) hide)
     )
-    (property "Datasheet" "~" (at 209.55 106.68 0)
+    (property "Datasheet" "10Ω 75V Thick Film 1%" (at 209.55 106.68 0)
       (effects (font (size 1.27 1.27)) hide)
     )
@@
       (effects (font (size 1.27 1.27)) hide)
     )
-    (property "Datasheet" "~" (at 209.55 73.66 0)
+    (property "Datasheet" "10Ω 75V Thick Film 1%" (at 209.55 73.66 0)
       (effects (font (size 1.27 1.27)) hide)
     )
@@
       (effects (font (size 1.27 1.27)))
     )
-    (property "Value" "0" (at 92.71 101.6 90)
+    (property "Value" "0R" (at 92.71 101.6 90)
       (effects (font (size 1.27 1.27)))
     )
@@
       (effects (font (size 1.27 1.27)) hide)
     )
-    (property "Datasheet" "~" (at 92.71 101.6 0)
+    (property "Datasheet" "0Ω 75V Thick Film 1%" (at 92.71 101.6 0)
       (effects (font (size 1.27 1.27)) hide)
     )
@@
       (effects (font (size 1.27 1.27)) hide)
     )
-    (property "Datasheet" "~" (at 209.55 109.22 0)
+    (property "Datasheet" "10Ω 75V Thick Film 1%" (at 209.55 109.22 0)
       (effects (font (size 1.27 1.27)) hide)
     )
@@
       (effects (font (size 1.27 1.27)) hide)
     )
-    (property "Datasheet" "~" (at 209.55 83.82 0)
+    (property "Datasheet" "10Ω 75V Thick Film 1%" (at 209.55 83.82 0)
       (effects (font (size 1.27 1.27)) hide)
     )
@@
       (effects (font (size 1.27 1.27)) hide)
     )
-    (property "Datasheet" "~" (at 209.55 76.2 0)
+    (property "Datasheet" "10Ω 75V Thick Film 1%" (at 209.55 76.2 0)
       (effects (font (size 1.27 1.27)) hide)
     )
@@
       (effects (font (size 1.27 1.27)))
     )
-    (property "Value" "100n" (at 111.76 45.72 90)
+    (property "Value" "100nF" (at 111.76 45.72 90)
       (effects (font (size 1.27 1.27)))
     )
@@
       (effects (font (size 1.27 1.27)) hide)
     )
-    (property "Datasheet" "~" (at 111.76 50.8 0)
+    (property "Datasheet" "100nF 50V X7R 10%" (at 111.76 50.8 0)
       (effects (font (size 1.27 1.27)) hide)
     )
@@
       (effects (font (size 1.27 1.27)) hide)
     )
-    (property "Datasheet" "~" (at 209.55 99.06 0)
-      (effects (font (size 1.27 1.27)) hide)
-    )
+    (property "Datasheet" "10Ω 75V Thick Film 1%" (at 209.55 99.06 0)
+      (effects (font (size 1.27 1.27)) hide)
+    )

Commit message: Assigned footprints for digital components
Parts:
- removed R107, R109, R111, R113, R114, R117, R118, R121: 10, Resistor_SMD:R_0603_1608Metric_Pad0.98x0.95mm_HandSolder, symbol Device:R
- removed R108, R112, R116, R120: 0R, Resistor_SMD:R_0603_1608Metric_Pad0.98x0.95mm_HandSolder, symbol Device:R
- added R27, R28, R30, R31, R32, R34, R35, R37: 10, Resistor_SMD:R_0603_1608Metric_Pad0.98x0.95mm_HandSolder, symbol Device:R
- U20, U22: value CDSOT236-T05 -> SRV05-4
- renumbered R106 to R86, R110 to R89, R115 to R93, R119 to R96
Connections:
- net DOUT1+: now also U20.1 (IO1), R27.2
- net DOUT1-: now also U20.3 (IO2), R28.2
- net DOUT2+: now also U20.4 (IO3), R30.2
- net DOUT2-: now also U20.6 (IO4), R31.2
- net DOUT3+: now also U22.1 (IO1), R32.2
- net DOUT3-: now also U22.3 (IO2), R34.2
- net DOUT4+: now also U22.4 (IO3), R35.2
- net DOUT4-: now also U22.6 (IO4), R37.2
- net at U21.11 (3Z): now also R34.1
- net at U21.6 (2Y): now also R30.1; no longer U20.4 (IO3)
- net at U21.5 (2Z): now also R31.1
- net at U21.3 (1Z): now also R28.1
- net at U21.10 (3Y): now also R32.1; no longer U22.1 (IO1)
- net at U21.14 (4Y): now also R35.1; no longer U22.4 (IO3)
- net at U21.13 (4Z): now also R37.1
- net at U21.2 (1Y): now also R27.1; no longer U20.1 (IO1)

Commit message: Redone power input circuit
Parts:
- renumbered C42 to C44, R27 to R26, R28 to R27, R30 to R29, R31 to R30, R32 to R31, R34 to R33, R35 to R34, R37 to R36, R86 to R85, R89 to R88, R93 to R92, R96 to R95, U20 to U21, U21 to U22, U22 to U23

Commit message: Optimized components by cost and footprint size
Parts:
- renumbered C44 to C42, R26 to R29, R27 to R30, R29 to R31, R30 to R32, R31 to R33, R33 to R34, R34 to R35, R88 to R86, R92 to R87, R95 to R88, U22 to U20, U23 to U22

Commit message: Excluded rare components
Parts:
- renumbered R29 to R31, R30 to R32, R31 to R33, R32 to R34, R33 to R35, R34 to R36, R35 to R37, R36 to R38, R85 to R87, R86 to R88, R87 to R89, R88 to R90

Commit message: Updated files to kicad 10
Parts:
- renumbered C42 to C37, R87 to R27, R88 to R28, R89 to R29, R90 to R30, U20 to U5, U21 to U6, U22 to U7
