File: receiver.kicad_sch (KiCad schematic)
At the start: 9 parts, among them J1 Conn_02x06_Odd_Even, J2 Conn_02x06_Odd_Even, J3 Conn_02x06_Odd_Even, J4 Conn_02x06_Odd_Even, J5 Conn_01x04, J6 Conn_02x06_Odd_Even, J7 Conn_02x12_Odd_Even, J8 Conn_02x06_Odd_Even, J9 Conn_02x06_Odd_Even

Commit message: Added annotations and missing footprints
Parts:
- J1, J2, J3, J4, J6, J8, J9: footprint (none) -> Connector_JST:JST_PHD_S12B-PHDSS_2x06_P2.00mm_Horizontal
- J5: footprint (none) -> Connector_PinHeader_2.54mm:PinHeader_1x04_P2.54mm_Vertical_SMD_Pin1Left
- J7: footprint (none) -> Connector_PinSocket_2.00mm:PinSocket_2x12_P2.00mm_Vertical
Other:
- sheet Ethernet 2 renamed Ethernet
- sheet Power Supply 2 renamed Power Supply
- moved on the sheet: J5, J6, J7

Commit message: Updated designators positions
Parts:
- renumbered J7 to J3, J3 to J4, J4 to J5, J5 to J6, J6 to J7
Changed lines of the file:
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@@
     (effects (font (size 3.048 3.048) (thickness 0.6096) bold) (justify left top))
   )
-  (text_box "Expansion header"
+  (text_box "Expansion socket"
     (at 76.2 254 0) (size 38.1 63.5)
     (stroke (width 0) (type default))
@@
   (symbol (lib_id "power:GND") (at 110.49 537.21 0) (unit 1)
     (in_bom yes) (on_board yes) (dnp no) (fields_autoplaced)
-    (property "Reference" "#PWR04" (at 110.49 543.56 0)
+    (property "Reference" "#PWR08" (at 110.49 543.56 0)
       (effects (font (size 1.27 1.27)) hide)
     )
@@
       (project "receiver"
         (path "/aa707d8b-0611-4fad-96c8-24f86e3803c6"
+          (reference "#PWR08") (unit 1)
+        )
+      )
+    )
+  )
+  (symbol (lib_id "power:+3V3") (at 81.28 459.74 0) (unit 1)
+    (in_bom yes) (on_board yes) (dnp no) (fields_autoplaced)
+    (property "Reference" "#PWR05" (at 81.28 463.55 0)
+      (effects (font (size 1.27 1.27)) hide)
+    )
+    (property "Value" "+3V3" (at 81.28 454.66 0)
+      (effects (font (size 1.27 1.27)))
+    )
+    (property "Footprint" "" (at 81.28 459.74 0)
+      (effects (font (size 1.27 1.27)) hide)
+    )
+    (property "Datasheet" "" (at 81.28 459.74 0)
+      (effects (font (size 1.27 1.27)) hide)
+    )
+    (pin "1")
+    (instances
+      (project "receiver"
+        (path "/aa707d8b-0611-4fad-96c8-24f86e3803c6"
+          (reference "#PWR05") (unit 1)
+        )
+      )
+    )
+  )
+  (symbol (lib_id "power:GND") (at 110.49 306.07 0) (unit 1)
+    (in_bom yes) (on_board yes) (dnp no) (fields_autoplaced)
+    (property "Reference" "#PWR04" (at 110.49 312.42 0)
+      (effects (font (size 1.27 1.27)) hide)
+    )
+    (property "Value" "GND" (at 110.49 311.15 0)
+      (effects (font (size 1.27 1.27)))
+    )
+    (property "Footprint" "" (at 110.49 306.07 0)
+      (effects (font (size 1.27 1.27)) hide)
+    )
+    (property "Datasheet" "" (at 110.49 306.07 0)
+      (effects (font (size 1.27 1.27)) hide)
+    )
+    (pin "1")
+    (instances
+      (project "receiver"
+        (path "/aa707d8b-0611-4fad-96c8-24f86e3803c6"
           (reference "#PWR04") (unit 1)
-        )
-      )
-    )
-  )
-  (symbol (lib_id "power:+3V3") (at 81.28 459.74 0) (unit 1)
-    (in_bom yes) (on_board yes) (dnp no) (fields_autoplaced)
-    (property "Reference" "#PWR01" (at 81.28 463.55 0)
-      (effects (font (size 1.27 1.27)) hide)
-    )
-    (property "Value" "+3V3" (at 81.28 454.66 0)
-      (effects (font (size 1.27 1.27)))
-    )
-    (property "Footprint" "" (at 81.28 459.74 0)
-      (effects (font (size 1.27 1.27)) hide)
-    )
-    (property "Datasheet" "" (at 81.28 459.74 0)
-      (effects (font (size 1.27 1.27)) hide)
-    )
-    (pin "1")
-    (instances
-      (project "receiver"
-        (path "/aa707d8b-0611-4fad-96c8-24f86e3803c6"
-          (reference "#PWR01") (unit 1)
-        )
-      )
-    )
-  )
-  (symbol (lib_id "power:GND") (at 110.49 306.07 0) (unit 1)
-    (in_bom yes) (on_board yes) (dnp no) (fields_autoplaced)
-    (property "Reference" "#PWR08" (at 110.49 312.42 0)
-      (effects (font (size 1.27 1.27)) hide)
-    )
-    (property "Value" "GND" (at 110.49 311.15 0)
-      (effects (font (size 1.27 1.27)))
-    )
-    (property "Footprint" "" (at 110.49 306.07 0)
-      (effects (font (size 1.27 1.27)) hide)
-    )
-    (property "Datasheet" "" (at 110.49 306.07 0)
-      (effects (font (size 1.27 1.27)) hide)
-    )
-    (pin "1")
-    (instances
-      (project "receiver"
-        (path "/aa707d8b-0611-4fad-96c8-24f86e3803c6"
-          (reference "#PWR08") (unit 1)
         )
       )
@@
   (symbol (lib_id "power:GND") (at 81.28 472.44 0) (unit 1)
     (in_bom yes) (on_board yes) (dnp no) (fields_autoplaced)
-    (property "Reference" "#PWR02" (at 81.28 478.79 0)
+    (property "Reference" "#PWR06" (at 81.28 478.79 0)
       (effects (font (size 1.27 1.27)) hide)
     )
@@
       (project "receiver"
         (path "/aa707d8b-0611-4fad-96c8-24f86e3803c6"
-          (reference "#PWR02") (unit 1)
+          (reference "#PWR06") (unit 1)
         )
       )
@@
   (symbol (lib_id "Connector_Generic:Conn_01x04") (at 99.06 464.82 0) (unit 1)
     (in_bom yes) (on_board yes) (dnp no) (fields_autoplaced)
-    (property "Reference" "J5" (at 101.6 464.82 0)
+    (property "Reference" "J6" (at 101.6 464.82 0)
       (effects (font (size 1.27 1.27)) (justify left))
     )
@@
       (project "receiver"
         (path "/aa707d8b-0611-4fad-96c8-24f86e3803c6"
-          (reference "J5") (unit 1)
+          (reference "J6") (unit 1)
         )
       )
@@
   (symbol (lib_id "Connector_Generic:Conn_02x06_Odd_Even") (at 93.98 529.59 0) (unit 1)
     (in_bom yes) (on_board yes) (dnp no) (fields_autoplaced)
-    (property "Reference" "J6" (at 95.25 518.16 0)
+    (property "Reference" "J7" (at 95.25 518.16 0)
       (effects (font (size 1.27 1.27)))
     )
@@
       (project "receiver"
         (path "/aa707d8b-0611-4fad-96c8-24f86e3803c6"
-          (reference "J6") (unit 1)
+          (reference "J7") (unit 1)
         )
       )
@@
   (symbol (lib_id "power:+5V") (at 80.01 524.51 0) (unit 1)
     (in_bom yes) (on_board yes) (dnp no) (fields_autoplaced)
-    (property "Reference" "#PWR03" (at 80.01 528.32 0)
+    (property "Reference" "#PWR07" (at 80.01 528.32 0)
       (effects (font (size 1.27 1.27)) hide)
     )
@@
       (project "receiver"
         (path "/aa707d8b-0611-4fad-96c8-24f86e3803c6"
-          (reference "#PWR03") (unit 1)
+          (reference "#PWR07") (unit 1)
         )
       )
@@
   (symbol (lib_id "power:GND") (at 80.01 306.07 0) (unit 1)
     (in_bom yes) (on_board yes) (dnp no) (fields_autoplaced)
-    (property "Reference" "#PWR07" (at 80.01 312.42 0)
+    (property "Reference" "#PWR03" (at 80.01 312.42 0)
       (effects (font (size 1.27 1.27)) hide)
     )
@@
       (project "receiver"
         (path "/aa707d8b-0611-4fad-96c8-24f86e3803c6"
-          (reference "#PWR07") (unit 1)
+          (reference "#PWR03") (unit 1)
         )
       )
@@
   (symbol (lib_id "Connector_Generic:Conn_02x06_Odd_Even") (at 474.98 373.38 0) (unit 1)
     (in_bom yes) (on_board yes) (dnp no) (fields_autoplaced)
-    (property "Reference" "J3" (at 476.25 361.95 0)
+    (property "Reference" "J4" (at 476.25 361.95 0)
       (effects (font (size 1.27 1.27)))
     )
@@
       (project "receiver"
         (path "/aa707d8b-0611-4fad-96c8-24f86e3803c6"
-          (reference "J3") (unit 1)
+          (reference "J4") (unit 1)
         )
       )
@@
   (symbol (lib_id "Connector_Generic:Conn_02x06_Odd_Even") (at 474.98 436.88 0) (unit 1)
     (in_bom yes) (on_board yes) (dnp no) (fields_autoplaced)
-    (property "Reference" "J4" (at 476.25 425.45 0)
+    (property "Reference" "J5" (at 476.25 425.45 0)
       (effects (font (size 1.27 1.27)))
     )
@@
       (project "receiver"
         (path "/aa707d8b-0611-4fad-96c8-24f86e3803c6"
-          (reference "J4") (unit 1)
+          (reference "J5") (unit 1)
         )
       )
@@
   (symbol (lib_id "power:+5V") (at 80.01 278.13 0) (unit 1)
     (in_bom yes) (on_board yes) (dnp no) (fields_autoplaced)
-    (property "Reference" "#PWR05" (at 80.01 281.94 0)
+    (property "Reference" "#PWR01" (at 80.01 281.94 0)
       (effects (font (size 1.27 1.27)) hide)
     )
@@
       (project "receiver"
         (path "/aa707d8b-0611-4fad-96c8-24f86e3803c6"
-          (reference "#PWR05") (unit 1)
+          (reference "#PWR01") (unit 1)
         )
       )
@@
   (symbol (lib_id "Connector_Generic:Conn_02x12_Odd_Even") (at 93.98 290.83 0) (unit 1)
     (in_bom yes) (on_board yes) (dnp no) (fields_autoplaced)
-    (property "Reference" "J7" (at 95.25 271.78 0)
+    (property "Reference" "J3" (at 95.25 271.78 0)
       (effects (font (size 1.27 1.27)))
     )
@@
       (project "receiver"
         (path "/aa707d8b-0611-4fad-96c8-24f86e3803c6"
-          (reference "J7") (unit 1)
+          (reference "J3") (unit 1)
         )
       )
@@
   (symbol (lib_id "power:+24V") (at 110.49 278.13 0) (unit 1)
     (in_bom yes) (on_board yes) (dnp no) (fields_autoplaced)
-    (property "Reference" "#PWR06" (at 110.49 281.94 0)
+    (property "Reference" "#PWR02" (at 110.49 281.94 0)
       (effects (font (size 1.27 1.27)) hide)
     )
@@
       (project "receiver"
         (path "/aa707d8b-0611-4fad-96c8-24f86e3803c6"
-          (reference "#PWR06") (unit 1)
-        )
-      )
+          (reference "#PWR02") (unit 1)
+        )
+      )

Commit message: Redone power input circuit
Parts:
- J1, J2, J4, J5, J7, J8, J9: value Conn_02x06_Odd_Even -> JST PHD B12B; footprint Connector_JST:JST_PHD_S12B-PHDSS_2x06_P2.00mm_Horizontal -> Connector_JST:JST_PHD_B12B-PHDSS_2x06_P2.00mm_Vertical
- J3: value Conn_02x12_Odd_Even -> Pin Socket
- J6: value Conn_01x04 -> JST PH B4B; footprint Connector_PinHeader_2.54mm:PinHeader_1x04_P2.54mm_Vertical_SMD_Pin1Left -> Connector_JST:JST_PH_B4B-PH-K_1x04_P2.00mm_Vertical
Changed lines of the file:
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@@
       (effects (font (size 1.27 1.27)))
     )
-    (property "Value" "Conn_02x06_Odd_Even" (at 476.25 618.49 0)
-      (effects (font (size 1.27 1.27)))
-    )
-    (property "Footprint" "Connector_JST:JST_PHD_S12B-PHDSS_2x06_P2.00mm_Horizontal" (at 474.98 627.38 0)
+    (property "Value" "JST PHD B12B" (at 476.25 618.49 0)
+      (effects (font (size 1.27 1.27)))
+    )
+    (property "Footprint" "Connector_JST:JST_PHD_B12B-PHDSS_2x06_P2.00mm_Vertical" (at 474.98 627.38 0)
       (effects (font (size 1.27 1.27)) hide)
     )
@@
       (effects (font (size 1.27 1.27)) (justify left))
     )
-    (property "Value" "Conn_01x04" (at 101.6 467.36 0)
+    (property "Value" "JST PH B4B" (at 101.6 467.36 0)
       (effects (font (size 1.27 1.27)) (justify left))
     )
-    (property "Footprint" "Connector_PinHeader_2.54mm:PinHeader_1x04_P2.54mm_Vertical_SMD_Pin1Left" (at 99.06 464.82 0)
+    (property "Footprint" "Connector_JST:JST_PH_B4B-PH-K_1x04_P2.00mm_Vertical" (at 99.06 464.82 0)
       (effects (font (size 1.27 1.27)) hide)
     )
@@
       (effects (font (size 1.27 1.27)))
     )
-    (property "Value" "Conn_02x06_Odd_Even" (at 476.25 554.99 0)
-      (effects (font (size 1.27 1.27)))
-    )
-    (property "Footprint" "Connector_JST:JST_PHD_S12B-PHDSS_2x06_P2.00mm_Horizontal" (at 474.98 563.88 0)
+    (property "Value" "JST PHD B12B" (at 476.25 554.99 0)
+      (effects (font (size 1.27 1.27)))
+    )
+    (property "Footprint" "Connector_JST:JST_PHD_B12B-PHDSS_2x06_P2.00mm_Vertical" (at 474.98 563.88 0)
       (effects (font (size 1.27 1.27)) hide)
     )
@@
       (effects (font (size 1.27 1.27)))
     )
-    (property "Value" "Conn_02x06_Odd_Even" (at 95.25 520.7 0)
-      (effects (font (size 1.27 1.27)))
-    )
-    (property "Footprint" "Connector_JST:JST_PHD_S12B-PHDSS_2x06_P2.00mm_Horizontal" (at 93.98 529.59 0)
+    (property "Value" "JST PHD B12B" (at 95.25 520.7 0)
+      (effects (font (size 1.27 1.27)))
+    )
+    (property "Footprint" "Connector_JST:JST_PHD_B12B-PHDSS_2x06_P2.00mm_Vertical" (at 93.98 529.59 0)
       (effects (font (size 1.27 1.27)) hide)
     )
@@
       (effects (font (size 1.27 1.27)))
     )
-    (property "Value" "Conn_02x06_Odd_Even" (at 476.25 173.99 0)
-      (effects (font (size 1.27 1.27)))
-    )
-    (property "Footprint" "Connector_JST:JST_PHD_S12B-PHDSS_2x06_P2.00mm_Horizontal" (at 474.98 182.88 0)
+    (property "Value" "JST PHD B12B" (at 476.25 173.99 0)
+      (effects (font (size 1.27 1.27)))
+    )
+    (property "Footprint" "Connector_JST:JST_PHD_B12B-PHDSS_2x06_P2.00mm_Vertical" (at 474.98 182.88 0)
       (effects (font (size 1.27 1.27)) hide)
     )
@@
       (effects (font (size 1.27 1.27)))
     )
-    (property "Value" "Conn_02x06_Odd_Even" (at 476.25 364.49 0)
-      (effects (font (size 1.27 1.27)))
-    )
-    (property "Footprint" "Connector_JST:JST_PHD_S12B-PHDSS_2x06_P2.00mm_Horizontal" (at 474.98 373.38 0)
+    (property "Value" "JST PHD B12B" (at 476.25 364.49 0)
+      (effects (font (size 1.27 1.27)))
+    )
+    (property "Footprint" "Connector_JST:JST_PHD_B12B-PHDSS_2x06_P2.00mm_Vertical" (at 474.98 373.38 0)
       (effects (font (size 1.27 1.27)) hide)
     )
@@
       (effects (font (size 1.27 1.27)))
     )
-    (property "Value" "Conn_02x06_Odd_Even" (at 476.25 427.99 0)
-      (effects (font (size 1.27 1.27)))
-    )
-    (property "Footprint" "Connector_JST:JST_PHD_S12B-PHDSS_2x06_P2.00mm_Horizontal" (at 474.98 436.88 0)
+    (property "Value" "JST PHD B12B" (at 476.25 427.99 0)
+      (effects (font (size 1.27 1.27)))
+    )
+    (property "Footprint" "Connector_JST:JST_PHD_B12B-PHDSS_2x06_P2.00mm_Vertical" (at 474.98 436.88 0)
       (effects (font (size 1.27 1.27)) hide)
     )
@@
       (effects (font (size 1.27 1.27)))
     )
-    (property "Value" "Conn_02x06_Odd_Even" (at 476.25 237.49 0)
-      (effects (font (size 1.27 1.27)))
-    )
-    (property "Footprint" "Connector_JST:JST_PHD_S12B-PHDSS_2x06_P2.00mm_Horizontal" (at 474.98 246.38 0)
+    (property "Value" "JST PHD B12B" (at 476.25 237.49 0)
+      (effects (font (size 1.27 1.27)))
+    )
+    (property "Footprint" "Connector_JST:JST_PHD_B12B-PHDSS_2x06_P2.00mm_Vertical" (at 474.98 246.38 0)
       (effects (font (size 1.27 1.27)) hide)
     )
@@
       (effects (font (size 1.27 1.27)))
     )
-    (property "Value" "Conn_02x12_Odd_Even" (at 95.25 274.32 0)
-      (effects (font (size 1.27 1.27)))
-    )
+    (property "Value" "Pin Socket" (at 95.25 274.32 0)
+      (effects (font (size 1.27 1.27)))
+    )

Commit message: Optimized components by cost and footprint size
Parts:
- removed J3: Pin Socket, Connector_PinSocket_2.00mm:PinSocket_2x12_P2.00mm_Vertical, symbol Connector_Generic:Conn_02x12_Odd_Even
- renumbered J7 to J1, J6 to J2, J1 to J3, J2 to J4, J4 to J5, J5 to J6, J8 to J7, J9 to J8
Connections:
- net SWDCLK: now also J2.2 (Pin_2); no longer J2.3 (Pin_3)
- net SWDIO: now also J2.3 (Pin_3); no longer J2.2 (Pin_2)
- no-connect marks 0 -> 14
