File: serializer.kicad_sch (KiCad schematic)
At the start: 26 parts, among them U1 STM32H723ZGT

Commit message: Updated files to kicad 10
Parts:
- renumbered C5 to C3, C3 to C4, C4 to C5
Other:
- moved on the sheet: C1, C10, C11, C12, C13, C14, C15, C16, C17, C18, C2, C3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
Changed lines of the file:
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@@
-(kicad_sch (version 20230121) (generator eeschema)
-  (paper "A4" portrait)
+(kicad_sch
+	(version 20260306)
+	(generator "eeschema")
+	(generator_version "10.0")
+	(paper "A3" portrait)
