File: analog_exp.kicad_pcb (KiCad board)
At the start: 2 copper layers, 229 parts, among them J10 HR911105A, J11 DC Barrel Jack, J2 JST PH S6B, J3 JST PH S6B, J4 JST PH S6B, J5 JST PH S6B, J6 JST PH S6B, J7 JST PH S6B, J8 JST PHD B12B, J9 JST PH B4B, U1 INA600B, U10 INA600B, U11 TPCDSOT236-T12, U12 INA600B, U13 INA600B, U14 TPCDSOT236-T12, U15 INA600B, U16 INA600B, U17 TPCDSOT236-T12, U18 INA600B, U19 TSB582, U2 TPCDSOT236-T12, U20 TSB582, U21 TSB582, U22 TSB582, U23 TSB582, U24 TSB582, U25 LAN8742AI, U26 LMR33630B, U27 TLV76733, U28 STM32H723ZGT, U3 INA600B, U4 INA600B, U5 TPCDSOT236-T12, U6 INA600B, U7 INA600B, U8 TPCDSOT236-T12, U9 INA600B, Y1 ABM8G-25MHz

Commit message: Updated power connector
Parts:
- removed J11: DC Barrel Jack, Connector_BarrelJack:BarrelJack_Horizontal
- added J1: Power MX 3.0, Connector_Molex:Molex_Micro-Fit_3.0_43045-0400_2x02_P3.00mm_Horizontal, F.Cu at (239.7, 68.5)
- moved J10 4.00 mm to (232.2, 91.9)
