File: ethernet.kicad_sch (KiCad schematic)
At the start: 32 parts, among them J10 HR911105A, U4 LAN8742AI, Y1 ABM8G-25MHz

Commit message: Excluded rare components
Parts:
- renumbered L4 to L3, R8 to R10, R9 to R11, R10 to R12, R11 to R13, R12 to R14, R13 to R15, R14 to R16, R15 to R17, R16 to R18, R17 to R19, R18 to R20, R19 to R21, R20 to R22, R21 to R23, R22 to R24, R23 to R25, R24 to R26, R7 to R9
Connections:
- net Earth is gone; now on net GND: J10.8, J10.SH

Commit message: Updated power connector
Parts:
- Y1: footprint Crystal:Crystal_SMD_3225-4Pin_3.2x2.5mm_HandSoldering -> Crystal:Crystal_SMD_3225-4Pin_3.2x2.5mm
Changed lines of the file:
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@@
 			)
 		)
-		(property "Footprint" "Crystal:Crystal_SMD_3225-4Pin_3.2x2.5mm_HandSoldering"
+		(property "Footprint" "Crystal:Crystal_SMD_3225-4Pin_3.2x2.5mm"
 			(at 80.01 124.46 0)
 			(hide yes)
